Commit message: Update joint limits

File: urdf/follower.urdf (robot description, URDF)
Before this commit: robot follower, 7 links, 6 joints
Joints:
- joint joint_1: limit lower=-3.14159265359 upper=3.14159265359 effort=0 velocity=0 -> lower=-2.4 upper=1.87 effort=0 velocity=0
- joint joint_2: limit lower=-3.14159265359 upper=3.14159265359 effort=0 velocity=0 -> lower=-1.86 upper=2.28 effort=0 velocity=0
- joint joint_3: limit lower=-3.14159265359 upper=3.14159265359 effort=0 velocity=0 -> lower=-2.42 upper=2.42 effort=0 velocity=0
- joint joint_4: limit lower=-3.14159265359 upper=3.14159265359 effort=0 velocity=0 -> lower=-1.93 upper=1.93 effort=0 velocity=0

File: urdf/leader.urdf (robot description, URDF)
Before this commit: robot leader, 7 links, 6 joints
Joints:
- joint joint_1: limit lower=-3.14159265359 upper=3.14159265359 effort=0 velocity=0 -> lower=-2.4 upper=1.87 effort=0 velocity=0
- joint joint_2: limit lower=-3.14159265359 upper=3.14159265359 effort=0 velocity=0 -> lower=-1.86 upper=2.28 effort=0 velocity=0
- joint joint_3: limit lower=-3.14159265359 upper=3.14159265359 effort=0 velocity=0 -> lower=-2.42 upper=2.42 effort=0 velocity=0
- joint joint_4: limit lower=-3.14159265359 upper=3.14159265359 effort=0 velocity=0 -> lower=-1.93 upper=1.93 effort=0 velocity=0
