Commit message: rename URDFs

File: trossen_arm_description/urdf/follower.urdf (robot description, URDF)
Before this commit: robot follower, 7 links, 6 joints
Links:
- link gripper: geometry collision mesh filename=package://trossen_arm_description/meshes/follower/gripper.s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; visual mesh filename=package://trossen_arm_description/meshes/follower/gripper.s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
- link link_1: geometry collision mesh filename=package://trossen_arm_description/meshes/follower/link_1.stl; visual mesh filename=package://trossen_arm_description/meshes/follower/link_1.stl
- link link_2: geometry collision mesh filename=package://trossen_arm_description/meshes/follower/link_2.stl; visual mesh filename=package://trossen_arm_description/meshes/follower/link_2.stl
- link link_3: geometry collision mesh filename=package://trossen_arm_description/meshes/follower/link_3.stl; visual mesh filename=package://trossen_arm_description/meshes/follower/link_3.stl
- link link_4: geometry collision mesh filename=package://trossen_arm_description/meshes/follower/link_4.stl; visual mesh filename=package://trossen_arm_description/meshes/follower/link_4.stl
- link link_5: geometry collision mesh filename=package://trossen_arm_description/meshes/follower/link_5.stl; visual mesh filename=package://trossen_arm_description/meshes/follower/link_5.stl

File: trossen_arm_description/urdf/leader.urdf (robot description, URDF)
Before this commit: robot leader, 7 links, 6 joints
Links:
- link base_link: geometry collision mesh filename=package://trossen_arm_description/meshes/leader/base_link.s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; visual mesh filename=package://trossen_arm_description/meshes/leader/base_link.s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
- link gripper: geometry collision mesh filename=package://trossen_arm_description/meshes/leader/gripper.stl; visual mesh filename=package://trossen_arm_description/meshes/leader/gripper.stl
- link link_1: geometry collision mesh filename=package://trossen_arm_description/meshes/leader/link_1.stl; visual mesh filename=package://trossen_arm_description/meshes/leader/link_1.stl
- link link_2: geometry collision mesh filename=package://trossen_arm_description/meshes/leader/link_2.stl; visual mesh filename=package://trossen_arm_description/meshes/leader/link_2.stl
- link link_3: geometry collision mesh filename=package://trossen_arm_description/meshes/leader/link_3.stl; visual mesh filename=package://trossen_arm_description/meshes/leader/link_3.stl
- link link_4: geometry collision mesh filename=package://trossen_arm_description/meshes/leader/link_4.stl; visual mesh filename=package://trossen_arm_description/meshes/leader/link_4.stl
- link link_5: geometry collision mesh filename=package://trossen_arm_description/meshes/leader/link_5.stl; visual mesh filename=package://trossen_arm_description/meshes/leader/link_5.stl
