Commit message: Update URDFs

File: trossen_arm_description/urdf/wxais_base.urdf (robot description, URDF)
Before this commit: robot wxai_leader, 9 links, 8 joints
Links:
- link base_link: geometry collision mesh filename=package://trossen_arm_description/meshes/wxais_base/base_li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; visual mesh filename=package://trossen_arm_description/meshes/wxais_base/base_li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
- link gripper_left: mass 0.07230515 -> 0.07618477; geometry collision mesh filename=package://trossen_arm_description/meshes/wxais_base/gripper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; visual mesh filename=package://trossen_arm_description/meshes/wxais_base/gripper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
- link gripper_right: mass 0.07230515 -> 0.07618477; geometry collision mesh filename=package://trossen_arm_description/meshes/wxais_base/gripper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; visual mesh filename=package://trossen_arm_description/meshes/wxais_base/gripper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
- link link_1: geometry collision mesh filename=package://trossen_arm_description/meshes/wxais_base/link_1.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; visual mesh filename=package://trossen_arm_description/meshes/wxais_base/link_1.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
- link link_2: geometry collision mesh filename=package://trossen_arm_description/meshes/wxais_base/link_2.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; visual mesh filename=package://trossen_arm_description/meshes/wxais_base/link_2.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
- link link_3: geometry collision mesh filename=package://trossen_arm_description/meshes/wxais_base/link_3.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; visual mesh filename=package://trossen_arm_description/meshes/wxais_base/link_3.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
- link link_4: geometry collision mesh filename=package://trossen_arm_description/meshes/wxais_base/link_4.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; visual mesh filename=package://trossen_arm_description/meshes/wxais_base/link_4.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
- link link_5: geometry collision mesh filename=package://trossen_arm_description/meshes/wxais_base/link_5.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; visual mesh filename=package://trossen_arm_description/meshes/wxais_base/link_5.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
- link link_6: mass 0.58782068 -> 0.51498747; geometry collision mesh filename=package://trossen_arm_description/meshes/wxais_base/link_6.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; visual mesh filename=package://trossen_arm_description/meshes/wxais_base/link_6.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
Joints:
- joint joint_0: limit lower=-3.14 upper=3.14 effort=0 velocity=0 -> lower=-3.14 upper=3.14 effort=27.0 velocity=3.14
- joint joint_1: axis 0 -1 0 -> 0 1 0; limit lower=-3.14 upper=3.14 effort=0 velocity=0 -> lower=0.0 upper=3.14 effort=27.0 velocity=3.14
- joint joint_2: limit lower=-3.14 upper=3.14 effort=0 velocity=0 -> lower=0.0 upper=2.356 effort=27.0 velocity=3.14
- joint joint_3: limit lower=-3.14 upper=3.14 effort=0 velocity=0 -> lower=-1.571 upper=1.571 effort=7.0 velocity=3.14
- joint joint_4: limit lower=-3.14 upper=3.14 effort=0 velocity=0 -> lower=-1.571 upper=1.571 effort=7.0 velocity=3.14
- joint joint_5: limit lower=-3.14 upper=3.14 effort=0 velocity=0 -> lower=-3.14 upper=3.14 effort=7.0 velocity=3.14
- joint joint_gl: limit lower=-3.14 upper=3.14 effort=0 velocity=0 -> lower=0 upper=0.044 effort=400.0 velocity=0.0875; origin xyz=0.078 0.01795 0 rpy=0 0 0 -> xyz=0.078 0.021375 0 rpy=0 0 0
- joint joint_gr: limit lower=-3.14 upper=3.14 effort=0 velocity=0 -> lower=-0.044 upper=0.0 effort=400.0 velocity=0.0875; origin xyz=0.078 -0.01795 0 rpy=0 0 0 -> xyz=0.078 -0.021375 0 rpy=0 0 0

File: trossen_arm_description/urdf/wxais_follower.urdf (robot description, URDF)
Before this commit: robot wxai_follower, 9 links, 8 joints
Links:
- link base_link: geometry collision mesh filename=package://trossen_arm_description/meshes/wxais_follower/bas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; visual mesh filename=package://trossen_arm_description/meshes/wxais_follower/bas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
- link gripper_left: geometry collision mesh filename=package://trossen_arm_description/meshes/wxais_follower/gri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; visual mesh filename=package://trossen_arm_description/meshes/wxais_follower/gri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
- link gripper_right: geometry collision mesh filename=package://trossen_arm_description/meshes/wxais_follower/gri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; visual mesh filename=package://trossen_arm_description/meshes/wxais_follower/gri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
- link link_1: geometry collision mesh filename=package://trossen_arm_description/meshes/wxais_follower/lin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; visual mesh filename=package://trossen_arm_description/meshes/wxais_follower/lin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
- link link_2: geometry collision mesh filename=package://trossen_arm_description/meshes/wxais_follower/lin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; visual mesh filename=package://trossen_arm_description/meshes/wxais_follower/lin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
- link link_3: geometry collision mesh filename=package://trossen_arm_description/meshes/wxais_follower/lin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; visual mesh filename=package://trossen_arm_description/meshes/wxais_follower/lin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
- link link_4: geometry collision mesh filename=package://trossen_arm_description/meshes/wxais_follower/lin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; visual mesh filename=package://trossen_arm_description/meshes/wxais_follower/lin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
- link link_5: geometry collision mesh filename=package://trossen_arm_description/meshes/wxais_follower/lin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; visual mesh filename=package://trossen_arm_description/meshes/wxais_follower/lin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
- link link_6: geometry collision mesh filename=package://trossen_arm_description/meshes/wxais_follower/lin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; visual mesh filename=package://trossen_arm_description/meshes/wxais_follower/lin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
Joints:
- joint joint_0: limit lower=-3.14 upper=3.14 effort=0 velocity=0 -> lower=-3.14 upper=3.14 effort=27.0 velocity=3.14
- joint joint_1: axis 0 -1 0 -> 0 1 0; limit lower=-3.14 upper=3.14 effort=0 velocity=0 -> lower=0.0 upper=2.356 effort=27.0 velocity=3.14
- joint joint_3: limit lower=-3.14 upper=3.14 effort=0 velocity=0 -> lower=-1.571 upper=1.571 effort=7.0 velocity=3.14
- joint joint_4: limit lower=-3.14 upper=3.14 effort=0 velocity=0 -> lower=-1.571 upper=1.571 effort=7.0 velocity=3.14
- joint joint_5: limit lower=-3.14 upper=3.14 effort=0 velocity=0 -> lower=-3.14 upper=3.14 effort=7.0 velocity=3.14
- joint joint_gl: limit lower=0 upper=0.05 effort=0 velocity=0 -> lower=0 upper=0.044 effort=400.0 velocity=0.0875
- joint joint_gr: limit lower=0 upper=0.05 effort=0 velocity=0 -> lower=-0.044 upper=0.0 effort=400.0 velocity=0.0875

File: trossen_arm_description/urdf/wxais_leader.urdf (robot description, URDF)
Before this commit: robot wxai_base, 9 links, 8 joints
Links:
- link base_link: geometry collision mesh filename=package://trossen_arm_description/meshes/wxais_leader/base_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; visual mesh filename=package://trossen_arm_description/meshes/wxais_leader/base_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
- link gripper_left: mass 0.07618477 -> 0.07230515; geometry collision mesh filename=package://trossen_arm_description/meshes/wxais_leader/gripp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; visual mesh filename=package://trossen_arm_description/meshes/wxais_leader/gripp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
- link gripper_right: mass 0.07618477 -> 0.07230515; geometry collision mesh filename=package://trossen_arm_description/meshes/wxais_leader/gripp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; visual mesh filename=package://trossen_arm_description/meshes/wxais_leader/gripp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
- link link_1: geometry collision mesh filename=package://trossen_arm_description/meshes/wxais_leader/link_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; visual mesh filename=package://trossen_arm_description/meshes/wxais_leader/link_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
- link link_2: geometry collision mesh filename=package://trossen_arm_description/meshes/wxais_leader/link_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; visual mesh filename=package://trossen_arm_description/meshes/wxais_leader/link_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
- link link_3: geometry collision mesh filename=package://trossen_arm_description/meshes/wxais_leader/link_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; visual mesh filename=package://trossen_arm_description/meshes/wxais_leader/link_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
- link link_4: geometry collision mesh filename=package://trossen_arm_description/meshes/wxais_leader/link_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; visual mesh filename=package://trossen_arm_description/meshes/wxais_leader/link_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
- link link_5: geometry collision mesh filename=package://trossen_arm_description/meshes/wxais_leader/link_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; visual mesh filename=package://trossen_arm_description/meshes/wxais_leader/link_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
- link link_6: mass 0.51498747 -> 0.58782068; geometry collision mesh filename=package://trossen_arm_description/meshes/wxais_leader/link_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; visual mesh filename=package://trossen_arm_description/meshes/wxais_leader/link_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
Joints:
- joint joint_0: limit lower=-3.14 upper=3.14 effort=0 velocity=0 -> lower=-3.14 upper=3.14 effort=27.0 velocity=3.14
- joint joint_1: axis 0 -1 0 -> 0 1 0; limit lower=-3.14 upper=3.14 effort=0 velocity=0 -> lower=0.0 upper=3.14 effort=27.0 velocity=3.14
- joint joint_2: limit lower=-3.14 upper=3.14 effort=0 velocity=0 -> lower=0.0 upper=2.356 effort=27.0 velocity=3.14
- joint joint_3: limit lower=-3.14 upper=3.14 effort=0 velocity=0 -> lower=-1.571 upper=1.571 effort=7.0 velocity=3.14
- joint joint_4: limit lower=-3.14 upper=3.14 effort=0 velocity=0 -> lower=-1.571 upper=1.571 effort=7.0 velocity=3.14
- joint joint_5: limit lower=-3.14 upper=3.14 effort=0 velocity=0 -> lower=-3.14 upper=3.14 effort=7.0 velocity=3.14
- joint joint_gl: limit lower=-3.14 upper=3.14 effort=0 velocity=0 -> lower=0 upper=0.044 effort=400.0 velocity=0.0875; origin xyz=0.078 0.021375 0 rpy=0 0 0 -> xyz=0.078 0.01795 0 rpy=0 0 0
- joint joint_gr: limit lower=-3.14 upper=3.14 effort=0 velocity=0 -> lower=-0.044 upper=0.0 effort=400.0 velocity=0.0875; origin xyz=0.078 -0.021375 0 rpy=0 0 0 -> xyz=0.078 -0.01795 0 rpy=0 0 0
