Commit message: Update masses, inertias

File: trossen_arm_description/urdf/wxai.urdf.xacro (robot description, xacro)
@@ -28,12 +28,12 @@
         xyz="-0.000375858292607297 -6.62873423389478E-05 0.027443162348488"
         rpy="0 0 0" />
-      <mass value="0.224120283282237" />
+      <mass value="0.45969858" />
       <inertia
-        ixx="7.35860325213388E-05"
-        ixy="-5.5802965495376E-09"
-        ixz="-1.09197878999961E-07"
-        iyy="7.09540647974691E-05"
-        iyz="2.83345191694863E-08"
-        izz="9.39810447747449E-05" />
+        ixx="0.00088006"
+        ixy="-0.00000011"
+        ixz="0.00000247"
+        iyy="0.00091243"
+        iyz="0.00000001"
+        izz="0.00021404" />
     </inertial>
     <visual>
@@ -62,12 +62,12 @@
         xyz="-0.000170717140750964 0.00142938385871949 0.0203939511450044"
         rpy="0 0 0" />
-      <mass value="0.151686278211385" />
+      <mass value="0.15270428" />
       <inertia
-        ixx="4.52732090013247E-05"
-        ixy="4.99255832155973E-09"
-        ixz="-5.2271534852903E-06"
-        iyy="3.79248659067107E-05"
-        iyz="1.71098662427643E-09"
-        izz="5.47838409636401E-05" />
+        ixx="0.00024937"
+        ixy="0.00000188"
+        ixz="0.00001402"
+        iyy="0.00014741"
+        iyz="0.00000665"
+        izz="0.00019264" />
     </inertial>
     <visual>
@@ -109,12 +109,12 @@
         xyz="-0.130142256375337 -0.00167447142265246 0.000487627804054119"
         rpy="0 0 0" />
-      <mass value="0.611815573610387" />
+      <mass value="1.15316319" />
       <inertia
-        ixx="0.000149806763097241"
-        ixy="-1.7277870445282E-10"
-        ixz="-3.38000453750262E-06"
-        iyy="0.00148729384708183"
-        iyz="2.31625560454475E-08"
-        izz="0.00144707829438896" />
+        ixx="0.00103625"
+        ixy="0.00044590"
+        ixz="-0.00000551"
+        iyy="0.03721553"
+        iyz="0.00000121"
+        izz="0.03780905" />
     </inertial>
     <visual>
@@ -156,12 +156,12 @@
         xyz="0.14889637986769 -0.000482795993009637 0.0533160727860036"
         rpy="0 0 0" />
-      <mass value="0.45269268333465" />
+      <mass value="0.68666638" />
       <inertia
-        ixx="0.000110975389841977"
-        ixy="-3.48101737443353E-09"
-        ixz="-3.07200929071728E-05"
-        iyy="0.000944180462979155"
-        iyz="6.93614969714099E-09"
-        izz="0.000877582982943938" />
+        ixx="0.00276824"
+        ixy="-0.00020811"
+        ixz="0.00741781"
+        iyy="0.03004807"
+        iyz="-0.00004748"
+        izz="0.02807083" />
     </inertial>
     <visual>
@@ -203,12 +203,12 @@
         xyz="0.0499341120147654 0.000395925820699807 0.0525216081324763"
         rpy="0 0 0" />
-      <mass value="0.255634517902238" />
+      <mass value="0.45789905" />
       <inertia
-        ixx="7.18320568805194E-05"
-        ixy="-1.13712805364293E-07"
-        ixz="-1.49801775716733E-05"
-        iyy="8.7280888805767E-05"
-        iyz="-2.74366918637329E-07"
-        izz="9.61155608615174E-05" />
+        ixx="0.00212398"
+        ixy="0.00000031"
+        ixz="0.00174386"
+        iyy="0.00378616"
+        iyz="0.00000007"
+        izz="0.00196042" />
     </inertial>
     <visual>
@@ -248,14 +248,14 @@
     <inertial>
       <origin
-        xyz="0.00680868461848289 -4.42257423186533E-05 -0.042030267777268"
-        rpy="0 0 0" />
-      <mass value="0.231616135893126" />
+        xyz="0.00412447 -0.00001138 -0.04283184"
+        rpy="0 0 0" />
+      <mass value="0.36693910" />
       <inertia
-        ixx="9.30059780887729E-05"
-        ixy="1.16427390931954E-08"
-        ixz="-5.56110087932421E-06"
-        iyy="7.3529063908031E-05"
-        iyz="2.17229329063081E-08"
-        izz="5.71912870238262E-05" />
+        ixx="0.00086230"
+        ixy="0.00000044"
+        ixz="-0.00006573"
+        iyy="0.00100004"
+        iyz="0.00000015"
+        izz="0.00027375" />
     </inertial>
     <visual>
@@ -297,12 +297,12 @@
         xyz="0.0454447042226515 -3.3312119305551E-05 6.37079439202992E-09"
         rpy="0 0 0" />
-      <mass value="0.303721927830436" />
+      <mass value="0.55469347" />
       <inertia
-        ixx="0.000265546503707589"
-        ixy="1.20149414530992E-08"
-        ixz="-1.90562961519435E-12"
-        iyy="7.41145702777998E-05"
-        iyz="2.20581201587785E-08"
-        izz="0.000225092515447716" />
+        ixx="0.00082429"
+        ixy="0.00000033"
+        ixz="0.00000026"
+        iyy="0.00164746"
+        iyz="-0.00000004"
+        izz="0.00224588" />
     </inertial>
     <visual>
@@ -328,5 +328,5 @@
   <joint name="joint_5" type="revolute">
     <origin
-      xyz="0.04095 0 -0.0455"
+      xyz="0.02895 0 -0.0455"
       rpy="0 0 0" />
     <parent link="link_5" />
@@ -344,12 +344,12 @@
         xyz="-0.0088960216342942 0.00403514361427389 0.00457900737971173"
         rpy="0 0 0" />
-      <mass value="0.0503630726101797" />
+      <mass value="0.05036313" />
       <inertia
-        ixx="1.05737957274845E-05"
-        ixy="1.46136484807991E-12"
-        ixz="3.60942349147469E-07"
-        iyy="3.3903119527156E-06"
-        iyz="3.14222250821931E-07"
-        izz="8.00539230293977E-06" />
+        ixx="0.00001923"
+        ixy="-0.00000345"
+        ixz="-0.00000309"
+        iyy="0.00001096"
+        iyz="0.00000265"
+        izz="0.00001858" />
     </inertial>
     <visual>
@@ -373,4 +373,17 @@
     </collision>
   </link>
+  <joint name="right_carriage_joint" type="prismatic">
+    <origin
+      xyz="0.0745 -0.023 0"
+      rpy="0 0 0" />
+    <parent link="link_6" />
+    <child link="carriage_right" />
+    <axis xyz="0 -1 0" />
+    <limit
+      lower="0"
+      upper="0"
+      effort="0"
+      velocity="0" />
+  </joint>
   <link name="carriage_left">
     <inertial>
@@ -378,12 +391,12 @@
         xyz="-0.00889602163429412 -0.00403515225638459 -0.00457907970794055"
         rpy="0 0 0" />
-      <mass value="0.0503630726101796" />
+      <mass value="0.05036313" />
       <inertia
-        ixx="1.05737957274845E-05"
-        ixy="1.46136486428222E-12"
-        ixz="-3.60957599947593E-07"
-        iyy="3.39031195271559E-06"
-        iyz="3.1422225082193E-07"
-        izz="8.00539230293976E-06" />
+        ixx="0.00001923"
+        ixy="0.00000345"
+        ixz="0.00000309"
+        iyy="0.00001096"
+        iyz="0.00000265"
+        izz="0.00001858" />
     </inertial>
     <visual>
@@ -420,17 +433,4 @@
       velocity="0" />
   </joint>
-  <joint name="right_carriage_joint" type="prismatic">
-    <origin
-      xyz="0.0745 -0.023 0"
-      rpy="0 0 0" />
-    <parent link="link_6" />
-    <child link="carriage_right" />
-    <axis xyz="0 -1 0" />
-    <limit
-      lower="0"
-      upper="0"
-      effort="0"
-      velocity="0" />
-  </joint>
   <xacro:if value="${variant == 'follower'}">
     <link name="camera_mount">
@@ -439,12 +439,12 @@
           xyz="0.0296855854757168 0.00562972530248117 0.0471179075194367"
           rpy="0 0 0" />
-        <mass value="0.0570755527903207" />
+        <mass value="0.04518012" />
         <inertia
-          ixx="2.20585029321409E-05"
-          ixy="7.68318500907665E-09"
-          ixz="-2.39739582889547E-06"
-          iyy="1.44836957156197E-05"
-          iyz="-2.0916223960996E-07"
-          izz="1.77235645161334E-05" />
+          ixx="0.00014960"
+          ixy="0.00000956"
+          ixz="0.00007148"
+          iyy="0.00017435"
+          iyz="0.00001857"
+          izz="0.00006808" />
       </inertial>
       <visual>
@@ -484,12 +484,13 @@
             xyz="0.0203255017535234 -0.00738697181677922 -0.081111420473222"
             rpy="0 0 0" />
-          <mass value="0.112693736705508" />
+          <mass value="0.05670184" />
           <inertia
-            ixx="0.000140625909869966"
-            ixy="-1.66988366454825E-07"
-            ixz="-1.11400669390463E-05"
-            iyy="0.000144172777491847"
-            iyz="-6.02779619964089E-06"
-            izz="1.67088155618759E-05" />
+            ixx="0.00042154"
+            ixy="-0.00000774"
+            ixz="-0.00008119"
+            iyy="0.00044231"
+            iyz="0.00003707"
+            izz="0.00003893"
+            />
         </inertial>
         <visual>
@@ -526,12 +527,12 @@
             xyz="0.00470472514618581 0.0029289423469383 -0.0226793519809421"
             rpy="0 0 0" />
-          <mass value="0.0334482861211268" />
+          <mass value="0.02647075" />
           <inertia
-            ixx="2.15521651819975E-05"
-            ixy="3.63797547113716E-07"
-            ixz="-1.57596838501154E-06"
-            iyy="2.02414918164589E-05"
-            iyz="2.57763866887699E-06"
-            izz="3.61328619227492E-06" />
+            ixx="0.00003230"
+            ixy="0.00000009"
+            ixz="-0.00000168"
+            iyy="0.00003143"
+            iyz="-0.00000390"
+            izz="0.00000380" />
         </inertial>
         <visual>
@@ -568,12 +569,12 @@
             xyz="-0.00139067941257306 -0.00434572084089531 -0.0280809769238789"
             rpy="0 0 0" />
-          <mass value="0.0226399376873522" />
+          <mass value="0.02088075" />
           <inertia
-            ixx="1.42933439011286E-05"
-            ixy="-4.47593635440579E-07"
-            ixz="-1.96106301547004E-06"
-            iyy="1.34809958328991E-05"
-            iyz="-1.88526807848634E-06"
-            izz="3.04977204952407E-06" />
+            ixx="0.00003399"
+            ixy="0.00000062"
+            ixz="0.00000315"
+            iyy="0.00003270"
+            iyz="0.00000479"
+            izz="0.00000358" />
         </inertial>
         <visual>
@@ -612,12 +613,12 @@
             xyz="0.0203252458247983 0.0073869167553635 -0.0811185578133218"
             rpy="0 0 0" />
-          <mass value="0.112678919461615" />
+          <mass value="0.05668184" />
           <inertia
-            ixx="0.000140599973264611"
-            ixy="1.67103682894012E-07"
-            ixz="-1.11380433253412E-05"
-            iyy="0.000144145877651198"
-            iyz="6.02862678704906E-06"
-            izz="1.67093313716455E-05" />
+            ixx="0.00042144"
+            ixy="0.00000773"
+            ixz="-0.00008117"
+            iyy="0.00044221"
+            iyz="-0.00003705"
+            izz="0.00003891" />
         </inertial>
         <visual>
@@ -654,12 +655,12 @@
             xyz="-0.00139125804767926 0.00434423906746726 -0.0280833807733366"
             rpy="0 0 0" />
-          <mass value="0.02263239368872" />
+          <mass value="0.02089075" />
           <inertia
-            ixx="1.4290610073001E-05"
-            ixy="4.47591482497247E-07"
-            ixz="-1.96065931243553E-06"
-            iyy="1.34803332199727E-05"
-            iyz="1.88505973329342E-06"
-            izz="3.04768339969034E-06" />
+            ixx="0.00003402"
+            ixy="-0.00000062"
+            ixz="0.00000315"
+            iyy="0.00003273"
+            iyz="-0.00000480"
+            izz="0.00000358" />
         </inertial>
         <visual>
@@ -696,12 +697,12 @@
             xyz="0.00470571265625336 -0.0029303338205246 -0.0226797825244652"
             rpy="0 0 0" />
-          <mass value="0.033440788167196" />
+          <mass value="0.02649075" />
           <inertia
-            ixx="2.15524335431287E-05"
-            ixy="-3.63973749098751E-07"
-            ixz="-1.57635074161868E-06"
-            iyy="2.02401286199949E-05"
-            iyz="-2.57756762041802E-06"
-            izz="3.61453863771449E-06" />
+            ixx="0.00003233"
+            ixy="-0.00000009"
+            ixz="-0.00000168"
+            iyy="0.00003146"
+            iyz="0.00000391"
+            izz="0.00000381" />
         </inertial>
         <visual>
@@ -741,12 +742,12 @@
           xyz="0.0188673477391189 -0.00900068987997303 -0.00215891070969232"
           rpy="0 0 0" />
-        <mass value="0.0316597159310581" />
+        <mass value="0.03090787" />
         <inertia
-          ixx="6.8727778392819E-06"
-          ixy="1.85875818408777E-06"
-          ixz="2.10469017580141E-07"
-          iyy="1.15019376101305E-05"
-          iyz="-1.42577971631089E-07"
-          izz="7.84951081816666E-06" />
+          ixx=" 0.00001034"
+          ixy="-0.00000849"
+          ixz="-0.00000155"
+          iyy="0.00002610"
+          iyz="0.00000080"
+          izz="0.00002544" />
       </inertial>
       <visual>
@@ -783,12 +784,12 @@
           xyz="0.0188673150206433 0.00900062850131636 -0.00215899211667148"
           rpy="0 0 0" />
-        <mass value="0.0316596868689633" />
+        <mass value="0.03090786" />
         <inertia
-          ixx="6.87278548212943E-06"
-          ixy="-1.85876231020021E-06"
-          ixz="2.10468320130317E-07"
-          iyy="1.15019142390085E-05"
-          iyz="1.42584910055048E-07"
-          izz="7.8494939350329E-06" />
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
Commit message: Add d405, rs2_desc dep

File: trossen_arm_description/urdf/wxai.urdf.xacro (robot description, xacro)
@@ -434,5 +434,5 @@
   </joint>
   <xacro:if value="${variant == 'follower'}">
-    <link name="camera_mount">
+    <link name="camera_mount_d405">
       <inertial>
         <origin
@@ -453,5 +453,5 @@
           rpy="0 0 0" />
         <geometry>
-          <mesh filename="${mesh_directory}/camera_mount.stl" />
+          <mesh filename="${mesh_directory}/camera_mount_d405.stl" />
         </geometry>
         <material name="">
@@ -464,5 +464,5 @@
           rpy="0 0 0" />
         <geometry>
-          <mesh filename="${mesh_directory}/camera_mount.stl" />
+          <mesh filename="${mesh_directory}/camera_mount_d405.stl" />
         </geometry>
       </collision>
@@ -473,7 +473,13 @@
         rpy="0 0 0" />
       <parent link="link_6" />
-      <child link="camera_mount" />
+      <child link="camera_mount_d405" />
       <axis xyz="0 0 0" />
     </joint>
+    <xacro:include filename="$(find realsense2_description)/urdf/_d405.urdf.xacro" />
+    <xacro:sensor_d405 parent="camera_mount_d405">
+      <origin
+        xyz="0.02927207801 0 0.03824951197"
+        rpy="0 ${radians(20)} 0" />
+    </xacro:sensor_d405>
   </xacro:if> <!-- variant == 'follower' -->
   <xacro:if value="${variant == 'leader'}">

Commit message: Add ee_gripper_link

File: trossen_arm_description/urdf/wxai.urdf.xacro (robot description, xacro)
@@ -826,4 +826,24 @@
       <axis xyz="0 0 0" />
     </joint>
+    <joint name="ee_gripper" type="fixed">
+      <origin
+        xyz="0.142 0 0"
+        rpy="0 0 0" />
+      <parent link="link_6" />
+      <child link="ee_gripper_link" />
+      <axis xyz="1 0 0" />
+    </joint>
+    <link name="ee_gripper_link">
+      <inertial>
+        <mass value="0.001"/>
+        <inertia
+          ixx="0.0001"
+          iyy="0.0001"
+          izz="0.0001"
+          ixy="0"
+          ixz="0"
+          iyz="0"/>
+      </inertial>
+    </link>
   </xacro:if> <!-- variant in ('base', 'follower') -->
 </robot>
