Commit message: Silence some warnings

File: trossen_arm_moveit/config/wxai.ros2_control.xacro (robot description, xacro)
@@ -2,5 +2,5 @@
 <robot xmlns:xacro="http://www.ros.org/wiki/xacro">
     <xacro:macro name="wxai_ros2_control" params="name initial_positions_file">
-        <xacro:property name="initial_positions" value="${load_yaml(initial_positions_file)['initial_positions']}"/>
+        <xacro:property name="initial_positions" value="${xacro.load_yaml(initial_positions_file)['initial_positions']}"/>
         <ros2_control name="${name}" type="system">
             <hardware>
@@ -13,6 +13,10 @@
                   <param name="initial_value">${initial_positions['joint_0']}</param>
                 </state_interface>
-                <state_interface name="velocity"/>
-                <state_interface name="effort"/>
+                <state_interface name="velocity">
+                  <param name="initial_value">0.0</param>
+                </state_interface>
+                <state_interface name="effort">
+                  <param name="initial_value">0.0</param>
+                </state_interface>
             </joint>
             <joint name="joint_1">
@@ -21,6 +25,10 @@
                   <param name="initial_value">${initial_positions['joint_1']}</param>
                 </state_interface>
-                <state_interface name="velocity"/>
-                <state_interface name="effort"/>
+                <state_interface name="velocity">
+                  <param name="initial_value">0.0</param>
+                </state_interface>
+                <state_interface name="effort">
+                  <param name="initial_value">0.0</param>
+                </state_interface>
             </joint>
             <joint name="joint_2">
@@ -29,6 +37,10 @@
                   <param name="initial_value">${initial_positions['joint_2']}</param>
                 </state_interface>
-                <state_interface name="velocity"/>
-                <state_interface name="effort"/>
+                <state_interface name="velocity">
+                  <param name="initial_value">0.0</param>
+                </state_interface>
+                <state_interface name="effort">
+                  <param name="initial_value">0.0</param>
+                </state_interface>
             </joint>
             <joint name="joint_3">
@@ -37,6 +49,10 @@
                   <param name="initial_value">${initial_positions['joint_3']}</param>
                 </state_interface>
-                <state_interface name="velocity"/>
-                <state_interface name="effort"/>
+                <state_interface name="velocity">
+                  <param name="initial_value">0.0</param>
+                </state_interface>
+                <state_interface name="effort">
+                  <param name="initial_value">0.0</param>
+                </state_interface>
             </joint>
             <joint name="joint_4">
@@ -45,6 +61,10 @@
                   <param name="initial_value">${initial_positions['joint_4']}</param>
                 </state_interface>
-                <state_interface name="velocity"/>
-                <state_interface name="effort"/>
+                <state_interface name="velocity">
+                  <param name="initial_value">0.0</param>
+                </state_interface>
+                <state_interface name="effort">
+                  <param name="initial_value">0.0</param>
+                </state_interface>
             </joint>
             <joint name="joint_5">
@@ -53,6 +73,10 @@
                   <param name="initial_value">${initial_positions['joint_5']}</param>
                 </state_interface>
-                <state_interface name="velocity"/>
-                <state_interface name="effort"/>
+                <state_interface name="velocity">
+                  <param name="initial_value">0.0</param>
+                </state_interface>
+                <state_interface name="effort">
+                  <param name="initial_value">0.0</param>
+                </state_interface>
             </joint>
         </ros2_control>
