Commit message: Add follower arm to MoveIt configs

File: trossen_arm_moveit/config/wxai.srdf.xacro (robot description, xacro)
@@ -4,5 +4,7 @@
     A URDF file must exist for this robot as well, where the joints and the links that are referenced are defined
 -->
-<robot name="wxai">
+<robot name="wxai" xmlns:xacro="http://ros.org/wiki/xacro">
+    <xacro:arg name="variant" default="base"/>        <!-- 'base', 'follower' -->
+    <xacro:property name="arm_variant" value="$(arg variant)"/>
     <!--GROUPS: Representation of a set of joints and links. This can be useful for specifying DOF to plan for, defining arms, end effectors, etc-->
     <!--LINKS: When a link is specified, the parent joint of that link (if it exists) is automatically included-->
@@ -90,3 +92,7 @@
     <disable_collisions link1="link_4" link2="link_6" reason="Never"/>
     <disable_collisions link1="link_5" link2="link_6" reason="Adjacent"/>
+    <xacro:if value="${arm_variant == 'follower'}">
+        <disable_collisions link1="camera_link" link2="camera_mount_d405" reason="Adjacent"/>
+        <disable_collisions link1="camera_mount_d405" link2="link_6" reason="Adjacent"/>
+    </xacro:if>  <!-- variant == 'follower' -->
 </robot>
