Commit message: cleanup

File: trossen_arm_description/urdf/ros2_control/wxai.ros2_control.xacro (robot description, xacro)
@@ -11,5 +11,5 @@
     </joint>
   </xacro:macro>
-  <xacro:macro name="wxai_ros2_control" params="name">
+  <xacro:macro name="wxai_ros2_control">
     <ros2_control name="TrossenArmHardwareInterface" type="system">
       <hardware>
@@ -29,4 +29,3 @@
     </ros2_control>
   </xacro:macro>
-  <xacro:wxai_ros2_control name="wxai"/>
 </robot>

File: trossen_arm_description/urdf/wxai.urdf.xacro (robot description, xacro)
@@ -14,4 +14,6 @@
   <xacro:property name="variant"                    value="$(arg variant)"/>
   <xacro:property name="arm_side"                   value="$(arg arm_side)"/>
+  <xacro:include filename="$(find trossen_arm_description)/urdf/ros2_control/wxai.ros2_control.xacro"/>
+  <xacro:wxai_ros2_control/>
   <xacro:if value="$(arg use_world_frame)">
     <link name="world"/>

Commit message: fake hardware in bringup

File: trossen_arm_description/urdf/ros2_control/wxai.ros2_control.xacro (robot description, xacro)
@@ -4,19 +4,30 @@
     <joint name="${name}">
       <command_interface name="position"/>
-      <!-- <command_interface name="velocity"/> -->
-      <!-- <command_interface name="effort"/> -->
-      <state_interface name="position"/>
-      <state_interface name="velocity"/>
-      <state_interface name="effort"/>
+      <state_interface name="position">
+          <param name="initial_value">0.0</param>
+      </state_interface>
+      <state_interface name="velocity">
+          <param name="initial_value">0.0</param>
+      </state_interface>
+      <state_interface name="effort">
+          <param name="initial_value">0.0</param>
+      </state_interface>
     </joint>
   </xacro:macro>
-  <xacro:macro name="wxai_ros2_control">
+  <xacro:macro name="wxai_ros2_control" params="use_fake_hardware">
     <ros2_control name="TrossenArmHardwareInterface" type="system">
-      <hardware>
-        <plugin>trossen_arm_hardware/TrossenArmHardwareInterface</plugin>
-        <param name="robot_model">0</param> <!-- 0: wxai_v0 -->
-        <param name="ip_address">192.168.1.2</param>
-        <param name="update_period">0.1</param>
-      </hardware>
+      <xacro:if value="$(arg use_fake_hardware)">
+        <hardware>
+          <plugin>fake_components/GenericSystem</plugin>
+        </hardware>
+      </xacro:if>  <!-- use_fake_hardware -->
+      <xacro:unless value="$(arg use_fake_hardware)">
+        <hardware>
+          <plugin>trossen_arm_hardware/TrossenArmHardwareInterface</plugin>
+          <param name="robot_model">0</param>        <!-- 0: wxai_v0 -->
+          <param name="ip_address">192.168.1.2</param>
+          <param name="update_period">0.1</param>
+        </hardware>
+      </xacro:unless>  <!-- use_fake_hardware -->
       <xacro:ros2_control_joint name="joint_0"/>
       <xacro:ros2_control_joint name="joint_1"/>

File: trossen_arm_description/urdf/wxai.urdf.xacro (robot description, xacro)
@@ -11,9 +11,10 @@
   <xacro:arg name="use_world_frame"                 default="false"/>     <!-- 'true', 'false' -->
   <xacro:arg name="base_link_frame"                 default="base_link"/>
+  <xacro:arg name="use_fake_hardware"               default="false"/>     <!-- 'true', 'false' -->
   <xacro:property name="mesh_directory"             value="package://trossen_arm_description/meshes/${robot_model}"/>
   <xacro:property name="variant"                    value="$(arg variant)"/>
   <xacro:property name="arm_side"                   value="$(arg arm_side)"/>
   <xacro:include filename="$(find trossen_arm_description)/urdf/ros2_control/wxai.ros2_control.xacro"/>
-  <xacro:wxai_ros2_control/>
+  <xacro:wxai_ros2_control use_fake_hardware="$(arg use_fake_hardware)"/>
   <xacro:if value="$(arg use_world_frame)">
     <link name="world"/>
